File: kvm-board.kicad_pcb (KiCad board)
At the start: 2 copper layers, 56 x 27 mm, 21 parts, among them J1 TYPE-C-31-M-12, J2 TYPE-C-31-M-12, U1 CH9329, U2 CH340N

Commit message: Move the Type-C pads to the rear of the connector
Rotate J1/J2 by 180 degrees and shift them outward so the SMT pads sit at the rear of the connector while the mouth stays at the board edge.  The CPL values for J1/J2 stay at 5.2/50.8 mm and 270/90 degrees.  U1/U2, D3/D4 and two caps move to keep the fanout routable; the CPL is updated for those parts.  DRC/ERC are clean.
Parts:
- moved C3 1.80 mm to (25.2, 11.5)
- moved J2 1.57 mm to (52.4, 14.0), turned to 90 degrees
- moved J1 1.57 mm to (3.63, 14.0), turned to -90 degrees
- moved D4 1.50 mm to (43.0, 13.5)
- moved U1 1.50 mm to (36.5, 14.0)
- moved U2 1.50 mm to (19.5, 14.0)
- moved D3 1.40 mm to (13.0, 13.5)
- moved C2 1.00 mm to (15.5, 17.5)
Routing:
- net VBUS_SER: track 29.2 -> 44.2 mm
- net USB_SER_DP: track 26.4 -> 13.1 mm, vias 2 -> 0
- net USB_SER_DM: track 25.7 -> 13.3 mm, vias 0 -> 3
- net VBUS_HID: track 29.9 -> 41.7 mm, vias 7 -> 5
- net USB_HID_DM: track 26.7 -> 15.8 mm, vias 2 -> 3
- net GND: track 18.8 -> 8.39 mm, vias 30 -> 28
- net USB_HID_DP: track 20.5 -> 11.9 mm, vias 3 -> 0
- net CC2_SER: track 14.8 -> 11.8 mm, vias 0 -> 2
- net UART_9329_TX: track 18.7 -> 15.7 mm
- net UART_9329_RX: track 18.7 -> 15.7 mm
- net +5V: track 75.3 -> 78.1 mm
- net LED_ACT: track 5.96 -> 8.46 mm
- net CC2_HID: track 14.8 -> 16.4 mm, vias 0 -> 2
- net V33: track 2.66 -> 4.20 mm
- net CC1_SER: track 11.3 -> 12.2 mm
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
Commit message: Fit the board outline to the published FRISK-CASE 3D model
Reshape the PCB to 65.4 x 31.4 mm with a 6.8 x 19.8 mm latch notch measured from the published FRISK_CASE1.stl, move J2 to the upper-right lobe, and swap D4's two identical USBLC6 channels so the J2 fanout stays planar. Regenerate the schematic, board images, gerbers, CPL and position files. DRC and ERC are clean.
Parts:
- moved R4 17.8 mm to (47.0, 3.75), turned to 0 degrees
- moved J2 12.7 mm to (61.8, 5.50)
- moved C7 11.1 mm to (55.0, 11.5)
- moved D4 9.97 mm to (52.0, 9.20)
- moved D2 1.15 mm to (53.1, 6.00)
- moved R3 0.81 mm to (47.0, 6.80), turned to 0 degrees
Connections:
- D4 pad 1: USB_HID_DP -> USB_HID_DM
- D4 pad 3: USB_HID_DM -> USB_HID_DP
- D4 pad 4: USB_HID_DM -> USB_HID_DP
- D4 pad 6: USB_HID_DP -> USB_HID_DM
Routing:
- net USB_HID_DP: track 11.9 -> 29.5 mm, vias 0 -> 4
- net USB_HID_DM: track 15.8 -> 30.2 mm, vias 3 -> 5
- net VBUS_HID: track 41.7 -> 31.1 mm, vias 5 -> 7
- net +5V: track 78.1 -> 79.3 mm
- net CC2_HID: track 16.4 -> 17.4 mm, vias 2 -> 0
- net CC1_HID: track 12.8 -> 13.6 mm, vias 0 -> 2
Other:
- board size 56 x 27 mm -> 65.4 x 31.4 mm
