File: serial-km-emulator.kicad_pcb (KiCad board)
At the start: 2 copper layers, 57.6 x 31.4 mm, 23 parts, among them J1 TYPE-C-31-M-12, J2 TYPE-C-31-M-12, U1 CH9329, U2 CH340N

Commit message: Rename the project to serial-km-emulator
Update the repository URL in the README and docs, regenerate the 41x41 silkscreen QR code (now 0.5 mm modules) and the top silkscreen title, and rename the KiCad project and fabrication files to match.
Other:
- board text added: "SERIAL-KM-EMULATOR CH9329EMU-USB replacement"
- board text removed: "KVM-BOARD CH9329EMU-USB replacement"
